File: hardware/miata-underglow.sch (KiCad schematic (older format))
At the start: 34 parts, among them J1 Micro_SD_Card, J2 FTDI, J3 LEDS, J4 CAN, Q1 SS8050, Q2 SS8050, U1 AMS1117-3.3, U2 TXS0108EPW, U3 AMS1117-5.0, U4 ESP32-WROOM-32D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

Commit message: Hardware Rev A
Parts:
- R3, R4: value R_Small -> 330
- R7: LCSC_PN C269754 -> C22107; Manufacturer Part Number RMC12061205%N -> 1206W4F1204T5E
Connections:
- net FTDI_RTS is gone; now on net FTDI_CTS: Q1.3 (E), R2.2
Changed lines of the file:
@@
 F 3 "~" H 10900 4050 50  0001 C CNN
 F 4 "1206" H 10900 4050 50  0001 C CNN "LCSC_FP"
-F 5 "C269754" H 10900 4050 50  0001 C CNN "LCSC_PN"
+F 5 "C22107" H 10900 4050 50  0001 C CNN "LCSC_PN"
 F 6 "" H 10900 4050 50  0001 C CNN "Field6"
-F 7 "RMC12061205%N" H 10900 4050 50  0001 C CNN "Manufacturer Part Number"
+F 7 "1206W4F1204T5E" H 10900 4050 50  0001 C CNN "Manufacturer Part Number"
 	1    10900 4050
 	1    0    0    -1
@@
 P 4300 900
 F 0 "R3" V 4104 900 50  0000 C CNN
-F 1 "R_Small" V 4195 900 50  0000 C CNN
+F 1 "330" V 4195 900 50  0000 C CNN
 F 2 "Resistor_SMD:R_0603_1608Metric" H 4300 900 50  0001 C CNN
 F 3 "~" H 4300 900 50  0001 C CNN
@@
 P 4300 1250
 F 0 "R4" V 4104 1250 50  0000 C CNN
-F 1 "R_Small" V 4195 1250 50  0000 C CNN
+F 1 "330" V 4195 1250 50  0000 C CNN
 F 2 "Resistor_SMD:R_0603_1608Metric" H 4300 1250 50  0001 C CNN
 F 3 "~" H 4300 1250 50  0001 C CNN
@@
 	1750 1750 1500 1750
 Text Label 1150 2150 0    50   ~ 0
-FTDI_RTS
+FTDI_CTS
 Wire Wire Line
 	1150 2150 1500 2150
 Text Label 650  2450 0    50   ~ 0
-FTDI_RTS
+FTDI_CTS
 Wire Wire Line
 	650  2450 1000 2450
